Commit message: installed urg_node and changed urdf to have correct frame links

File: yeetbot_navigation/urdf/pioneer3at.urdf.xacro (robot description, xacro)
@@ -154,5 +154,5 @@
 	</joint>
 <!-- Kinect Depth Sensor  -->
-     <link name="kinect_link">
+     <link name="camera_link">
           <visual>
             <geometry>
@@ -169,10 +169,10 @@
           </inertial>
         </link>
-        <joint name="base_kinect_joint" type="fixed">
+        <joint name="base_camera_joint" type="fixed">
                 <origin xyz="0.2 0 1.193" rpy="0 0 0"/>
                 <parent link="base_link"/>
-                <child link="kinect_link"/>
+                <child link="camera_link"/>
         </joint>
-        <link name="kinect_depth_frame">
+        <link name="camera_depth_frame">
           <inertial>
               <mass value="0.0001" />
@@ -183,10 +183,10 @@
           </inertial>
         </link>
-        <joint name="kinect_depth_joint" type="fixed">
+        <joint name="camera_depth_joint" type="fixed">
           <origin xyz="0 0.028 0" rpy="0 0 0" />
-          <parent link="kinect_link" />
-          <child link="kinect_depth_frame" />
+          <parent link="camera_link" />
+          <child link="camera_depth_frame" />
         </joint>
-        <link name="kinect_depth_optical_frame">
+        <link name="camera_depth_optical_frame">
           <inertial>
               <mass value="0.0001" />
@@ -199,6 +199,6 @@
         <joint name="depth_optical_joint" type="fixed">
           <origin xyz="0 0 0" rpy="${pi/2} 0 ${pi/2}" />
-          <parent link="kinect_depth_frame" />
-          <child link="kinect_depth_optical_frame" />
+          <parent link="camera_depth_frame" />
+          <child link="camera_depth_optical_frame" />
         </joint>
 <!-- Hokuyo LIDAR -->
@@ -216,5 +216,5 @@
                 <child link="lidar_link"/>
         </joint>
-	<link name="beam_link">
+	<link name="laser">
           <inertial>
               <mass value="0.0001" />
@@ -225,8 +225,8 @@
           </inertial>
 	</link>
-        <joint name="lidar_beam_joint" type="fixed">
+        <joint name="lidar_laser_joint" type="fixed">
                 <origin xyz="0 0 -0.0225" rpy="${pi} 0 0"/>
                 <parent link="lidar_link"/>
-                <child link="beam_link"/>
+                <child link="laser"/>
         </joint>
 <xacro:macro name="p3at_drive_side" params="side reflect">

Commit message: added launch file that works most of the time

File: yeetbot_navigation/urdf/pioneer3at.urdf.xacro (robot description, xacro)
@@ -69,4 +69,59 @@
 		<child link="top_plate"/>
 	</joint>
+<!-- Lidar Holder -->
+	<link name="lidar_holder">
+		<inertial>
+			<mass value="0.05"/>
+			<origin xyz="-0.025 0 -0.223"/>
+			<inertia ixx="1.0" ixy="0.0" ixz="0.0"
+				 iyy="1.0" iyz="0.0"
+ 				izz="1.0"/>
+		</inertial>
+		<visual>
+			<origin xyz="0 0 0" rpy="0 0 0"/>
+			<geometry name="pioneer_geom">
+				<mesh filename="package://yeetbot_navigation/meshes/lidar_holder.STL" scale="0.001 0.001 0.001"/>
+			</geometry>
+			<material name="TopBlack">
+					<color rgba="0.038 0.038 0.038 1.0"/>
+			</material>
+		</visual>
+	</link>
+	<gazebo reference="lidar_holder">
+	    <material>Gazebo/Black</material>
+	</gazebo>
+	<joint name="top_lh_joint" type="fixed">
+		<origin xyz="0.109 -0.195 0.003" rpy="0 0 0"/>
+		<parent link="top_plate"/>
+		<child link="lidar_holder"/>
+	</joint>
+<!-- Hokuyo LIDAR -->
+	<link name="lidar_link">
+	<visual>
+		<geometry>
+			<box size="0.05 0.05 0.07" />
+		</geometry>
+		<material name="Green"/>
+	</visual>
+	</link>
+        <joint name="lh_lidar_joint" type="fixed">
+                <origin xyz="0.172 0.195 -0.035" rpy="0 0 0"/>
+                <parent link="lidar_holder"/>
+                <child link="lidar_link"/>
+        </joint>
+	<link name="laser">
+          <inertial>
+              <mass value="0.0001" />
+              <origin xyz="0 0 0" />
+              <inertia ixx="0.0001" ixy="0.0" ixz="0.0"
+                       iyy="0.0001" iyz="0.0"
+                       izz="0.0001" />
+          </inertial>
+	</link>
+        <joint name="lidar_laser_joint" type="fixed">
+                <origin xyz="0 0 -0.0225" rpy="${pi} 0 0"/>
+                <parent link="lidar_link"/>
+                <child link="laser"/>
+        </joint>
 <!-- Drawer Frame -->
 	<link name="drawer_frame">
@@ -101,55 +156,4 @@
 		<parent link="top_plate"/>
 		<child link="drawer_frame"/>
-	</joint>
-<!-- Front + Back Sonar -->
-	<link name="front_sonar">
-		<inertial>
-			<mass value="0.1"/>
-			<origin xyz="0 0 0"/>
-			<inertia ixx="1.0" ixy="0.0" ixz="0.0"
-				 iyy="1.0" iyz="0.0" izz="1.0"/>
-		</inertial>
-		<visual>
-			<origin xyz="0 0 0" rpy="0 0 0"/>
-			<geometry name="pioneer_geom">
-				<mesh filename="package://yeetbot_navigation/meshes/front_sonar.stl"/>
-			</geometry>
-			<material name="SonarYellow">
-				<color rgba="0.715 0.583 0.210 1.0"/>
-			</material>
-		</visual>
-	</link>
-	<gazebo reference="front_sonar">
-		<material value="Gazebo/Yellow"/>
-	</gazebo>
-	<joint name="base_front_joint" type="fixed">
-		<origin xyz="0.193 0 0.25" rpy="0 0 0"/>
-		<parent link="base_link"/>
-		<child link="front_sonar"/>
-	</joint>
-	<link name="back_sonar">
-		<inertial>
-			<mass value="0.1"/>
-			<origin xyz="0 0 0"/>
-			<inertia ixx="1.0" ixy="0.0" ixz="0.0"
-				 iyy="1.0" iyz="0.0" izz="1.0"/>
-		</inertial>
-		<visual>
-			<origin xyz="0 0 0" rpy="0 0 0"/>
-			<geometry name="pioneer_geom">
-				<mesh filename="package://yeetbot_navigation/meshes/back_sonar.stl"/>
-			</geometry>
-			<material name="SonarYellow">
-				<color rgba="0.715 0.583 0.210 1.0"/>
-			</material>
-		</visual>
-	</link>
-	<gazebo reference="back_sonar">
-		<material value="Gazebo/Yellow"/>
-	</gazebo>
-	<joint name="base_back_joint" type="fixed">
-		<origin xyz="-0.187 0 0.247" rpy="0 0 0"/>
-		<parent link="base_link"/>
-		<child link="back_sonar"/>
 	</joint>
 <!-- Kinect Depth Sensor  -->
@@ -169,7 +173,7 @@
           </inertial>
         </link>
-        <joint name="base_camera_joint" type="fixed">
-                <origin xyz="0.2 0 1.193" rpy="0 0 0"/>
-                <parent link="base_link"/>
+        <joint name="frame_camera_joint" type="fixed">
+                <origin xyz="0.122 0.916 0.05" rpy="${pi * 1.5} ${pi * 0.5} 0"/>
+                <parent link="drawer_frame"/>
                 <child link="camera_link"/>
         </joint>
@@ -202,32 +206,55 @@
           <child link="camera_depth_optical_frame" />
         </joint>
-<!-- Hokuyo LIDAR -->
-	<link name="lidar_link">
-	<visual>
-		<geometry>
-			<box size="0.05 0.05 0.07" />
-		</geometry>
-		<material name="Green"/>
-	</visual>
-	</link>
-        <joint name="base_lidar_joint" type="fixed">
-                <origin xyz="0.285 0 0.235" rpy="0 0 0"/>
-                <parent link="base_link"/>
-                <child link="lidar_link"/>
-        </joint>
-	<link name="laser">
-          <inertial>
-              <mass value="0.0001" />
-              <origin xyz="0 0 0" />
-              <inertia ixx="0.0001" ixy="0.0" ixz="0.0"
-                       iyy="0.0001" iyz="0.0"
-                       izz="0.0001" />
-          </inertial>
-	</link>
-        <joint name="lidar_laser_joint" type="fixed">
-                <origin xyz="0 0 -0.0225" rpy="${pi} 0 0"/>
-                <parent link="lidar_link"/>
-                <child link="laser"/>
-        </joint>
+<!-- Front + Back Sonar -->
+	<link name="front_sonar">
+		<inertial>
+			<mass value="0.1"/>
+			<origin xyz="0 0 0"/>
+			<inertia ixx="1.0" ixy="0.0" ixz="0.0"
+				 iyy="1.0" iyz="0.0" izz="1.0"/>
+		</inertial>
+		<visual>
+			<origin xyz="0 0 0" rpy="0 0 0"/>
+			<geometry name="pioneer_geom">
+				<mesh filename="package://yeetbot_navigation/meshes/front_sonar.stl"/>
+			</geometry>
+			<material name="SonarYellow">
+				<color rgba="0.715 0.583 0.210 1.0"/>
+			</material>
+		</visual>
+	</link>
+	<gazebo reference="front_sonar">
+		<material value="Gazebo/Yellow"/>
+	</gazebo>
+	<joint name="base_front_joint" type="fixed">
+		<origin xyz="0.193 0 0.25" rpy="0 0 0"/>
+		<parent link="base_link"/>
+		<child link="front_sonar"/>
+	</joint>
+	<link name="back_sonar">
+		<inertial>
+			<mass value="0.1"/>
+			<origin xyz="0 0 0"/>
+			<inertia ixx="1.0" ixy="0.0" ixz="0.0"
+				 iyy="1.0" iyz="0.0" izz="1.0"/>
+		</inertial>
+		<visual>
+			<origin xyz="0 0 0" rpy="0 0 0"/>
+			<geometry name="pioneer_geom">
+				<mesh filename="package://yeetbot_navigation/meshes/back_sonar.stl"/>
+			</geometry>
+			<material name="SonarYellow">
+				<color rgba="0.715 0.583 0.210 1.0"/>
+			</material>
+		</visual>
+	</link>
+	<gazebo reference="back_sonar">
+		<material value="Gazebo/Yellow"/>
+	</gazebo>
+	<joint name="base_back_joint" type="fixed">
+		<origin xyz="-0.187 0 0.247" rpy="0 0 0"/>
+		<parent link="base_link"/>
+		<child link="back_sonar"/>
+	</joint>
 <xacro:macro name="p3at_drive_side" params="side reflect">
   <!-- Front Axles + Wheels + Hubcaps -->

Commit message: yeet nav again

File: yeetbot_navigation/urdf/pioneer3at.urdf.xacro (robot description, xacro)
@@ -173,9 +173,13 @@
           </inertial>
         </link>
-        <joint name="frame_camera_joint" type="fixed">
-                <origin xyz="0.122 0.916 0.05" rpy="${pi * 1.5} ${pi * 0.5} 0"/>
-                <parent link="drawer_frame"/>
+	<joint name="base_camera_joint" type="revolute">
+  	<axis xyz="0 1 0"/>
+    <anchor xyz="0 0 0"/>
+    <limit effort="100" velocity="100" lower="${pi*-0.5}" upper="${pi*0.5}"/>
+    <joint_properties damping="0.7"/>
+                <origin xyz="0.2 0 1.193" rpy="${pi} 0 0"/>
+                <parent link="base_link"/>
                 <child link="camera_link"/>
-        </joint>
+	</joint>
         <link name="camera_depth_frame">
           <inertial>

Commit message: testing dwa

File: yeetbot_navigation/urdf/pioneer3at.urdf.xacro (robot description, xacro)
@@ -157,4 +157,81 @@
 		<child link="drawer_frame"/>
 	</joint>
+<!-- april tags-->
+     <link name="yeet_box">
+          <visual>
+            <geometry>
+              <box size="0.21 0.21 0.21" />
+            </geometry>
+            <material name="Blue" />
+          </visual>
+          <inertial>
+              <mass value="0.0001" />
+              <origin xyz="0 0 0" />
+              <inertia ixx="0.0001" ixy="0.0" ixz="0.0"
+                       iyy="0.0001" iyz="0.0"
+                       izz="0.0001" />
+          </inertial>
+        </link>
+        <joint name="base_yeet_joint" type="fixed">
+                <origin xyz="0 0 1.28" rpy="0 0 0"/>
+                <parent link="base_link"/>
+                <child link="yeet_box"/>
+        </joint>
+     <link name="tag0">
+          <inertial>
+              <mass value="0.0001" />
+              <origin xyz="0 0 0" />
+              <inertia ixx="0.0001" ixy="0.0" ixz="0.0"
+                       iyy="0.0001" iyz="0.0"
+                       izz="0.0001" />
+          </inertial>
+        </link>
+        <joint name="yeet_tag0_joint" type="fixed">
+                <origin xyz="0 -0.105 0" rpy="${pi*0.5} 0 0"/>
+                <parent link="yeet_box"/>
+                <child link="tag0"/>
+        </joint>
+     <link name="tag1">
+          <inertial>
+              <mass value="0.0001" />
+              <origin xyz="0 0 0" />
+              <inertia ixx="0.0001" ixy="0.0" ixz="0.0"
+                       iyy="0.0001" iyz="0.0"
+                       izz="0.0001" />
+          </inertial>
+        </link>
+        <joint name="yeet_tag1_joint" type="fixed">
+                <origin xyz="-0.105 0 0" rpy="${pi*0.5} 0 ${pi*1.5}"/>
+                <parent link="yeet_box"/>
+                <child link="tag1"/>
+        </joint>
+     <link name="tag2">
+          <inertial>
+              <mass value="0.0001" />
+              <origin xyz="0 0 0" />
+              <inertia ixx="0.0001" ixy="0.0" ixz="0.0"
+                       iyy="0.0001" iyz="0.0"
+                       izz="0.0001" />
+          </inertial>
+        </link>
+        <joint name="yeet_tag2_joint" type="fixed">
+                <origin xyz="0 0.105 0" rpy="${pi * 1.5} ${pi} 0"/>
+                <parent link="yeet_box"/>
+                <child link="tag2"/>
+        </joint>
+     <link name="tag3">
+          <inertial>
+              <mass value="0.0001" />
+              <origin xyz="0 0 0" />
+              <inertia ixx="0.0001" ixy="0.0" ixz="0.0"
+                       iyy="0.0001" iyz="0.0"
+                       izz="0.0001" />
+          </inertial>
+        </link>
+        <joint name="yeet_tag3_joint" type="fixed">
+                <origin xyz="0.105 0 0" rpy="${pi * 0.5} 0 ${pi * 0.5}"/>
+                <parent link="yeet_box"/>
+                <child link="tag3"/>
+        </joint>
 <!-- Kinect Depth Sensor  -->
      <link name="camera_link">

Commit message: add april tags to urdf

File: yeetbot_navigation/urdf/pioneer3at.urdf.xacro (robot description, xacro)
@@ -157,4 +157,82 @@
 		<child link="drawer_frame"/>
 	</joint>
+<!-- april tags-->
+174      <link name="yeet_box">
+175           <visual>
+176             <geometry>
+177               <box size="0.21 0.21 0.21" />
+178             </geometry>
+179             <material name="Blue" />
+180           </visual>
+181           <inertial>
+182               <mass value="0.0001" />
+183               <origin xyz="0 0 0" />
+184               <inertia ixx="0.0001" ixy="0.0" ixz="0.0"
+185                        iyy="0.0001" iyz="0.0"
+186                        izz="0.0001" />
+187           </inertial>
+188         </link>
+189         <joint name="base_yeet_joint" type="fixed">
+190                 <origin xyz="0 0 1.28" rpy="0 0 0"/>
+191                 <parent link="base_link"/>
+192                 <child link="yeet_box"/>
+193         </joint>
+194
+195      <link name="tag0">
+196           <inertial>
+197               <mass value="0.0001" />
+198               <origin xyz="0 0 0" />
+199               <inertia ixx="0.0001" ixy="0.0" ixz="0.0"
+200                        iyy="0.0001" iyz="0.0"
+201                        izz="0.0001" />
+202           </inertial>
+203         </link>
+204         <joint name="yeet_tag0_joint" type="fixed">
+205                 <origin xyz="0 -0.105 0" rpy="${pi*0.5} 0 0"/>
+206                 <parent link="yeet_box"/>
+207                 <child link="tag0"/>
+208         </joint>
+209      <link name="tag1">
+210           <inertial>
+211               <mass value="0.0001" />
+212               <origin xyz="0 0 0" />
+213               <inertia ixx="0.0001" ixy="0.0" ixz="0.0"
+214                        iyy="0.0001" iyz="0.0"
+215                        izz="0.0001" />
+216           </inertial>
+217         </link>
+218         <joint name="yeet_tag1_joint" type="fixed">
+219                 <origin xyz="-0.105 0 0" rpy="${pi*0.5} 0 ${pi*1.5}"/>
+220                 <parent link="yeet_box"/>
+221                 <child link="tag1"/>
+222         </joint>
+223      <link name="tag2">
+224           <inertial>
+225               <mass value="0.0001" />
+226               <origin xyz="0 0 0" />
+227               <inertia ixx="0.0001" ixy="0.0" ixz="0.0"
+228                        iyy="0.0001" iyz="0.0"
+229                        izz="0.0001" />
+230           </inertial>
+231         </link>
+232         <joint name="yeet_tag2_joint" type="fixed">
+233                 <origin xyz="0 0.105 0" rpy="${pi * 1.5} ${pi} 0"/>
+234                 <parent link="yeet_box"/>
+235                 <child link="tag2"/>
+236         </joint>
+237      <link name="tag3">
+238           <inertial>
+239               <mass value="0.0001" />
+240               <origin xyz="0 0 0" />
+241               <inertia ixx="0.0001" ixy="0.0" ixz="0.0"
+242                        iyy="0.0001" iyz="0.0"
+243                        izz="0.0001" />
+244           </inertial>
+245         </link>
+246         <joint name="yeet_tag3_joint" type="fixed">
+247                 <origin xyz="0.105 0 0" rpy="${pi * 0.5} 0 ${pi * 0.5}"/>
+248                 <parent link="yeet_box"/>
+249                 <child link="tag3"/>
+250         </joint>
 <!-- Kinect Depth Sensor  -->
      <link name="camera_link">

Commit message: urdf fix, movebase no static map transform

File: yeetbot_navigation/urdf/pioneer3at.urdf.xacro (robot description, xacro)
@@ -158,81 +158,80 @@
 	</joint>
 <!-- april tags-->
-174      <link name="yeet_box">
-175           <visual>
-176             <geometry>
-177               <box size="0.21 0.21 0.21" />
-178             </geometry>
-179             <material name="Blue" />
-180           </visual>
-181           <inertial>
-182               <mass value="0.0001" />
-183               <origin xyz="0 0 0" />
-184               <inertia ixx="0.0001" ixy="0.0" ixz="0.0"
-185                        iyy="0.0001" iyz="0.0"
-186                        izz="0.0001" />
-187           </inertial>
-188         </link>
-189         <joint name="base_yeet_joint" type="fixed">
-190                 <origin xyz="0 0 1.28" rpy="0 0 0"/>
-191                 <parent link="base_link"/>
-192                 <child link="yeet_box"/>
-193         </joint>
-194
-195      <link name="tag0">
-196           <inertial>
-197               <mass value="0.0001" />
-198               <origin xyz="0 0 0" />
-199               <inertia ixx="0.0001" ixy="0.0" ixz="0.0"
-200                        iyy="0.0001" iyz="0.0"
-201                        izz="0.0001" />
-202           </inertial>
-203         </link>
-204         <joint name="yeet_tag0_joint" type="fixed">
-205                 <origin xyz="0 -0.105 0" rpy="${pi*0.5} 0 0"/>
-206                 <parent link="yeet_box"/>
-207                 <child link="tag0"/>
-208         </joint>
-209      <link name="tag1">
-210           <inertial>
-211               <mass value="0.0001" />
-212               <origin xyz="0 0 0" />
-213               <inertia ixx="0.0001" ixy="0.0" ixz="0.0"
-214                        iyy="0.0001" iyz="0.0"
-215                        izz="0.0001" />
-216           </inertial>
-217         </link>
-218         <joint name="yeet_tag1_joint" type="fixed">
-219                 <origin xyz="-0.105 0 0" rpy="${pi*0.5} 0 ${pi*1.5}"/>
-220                 <parent link="yeet_box"/>
-221                 <child link="tag1"/>
-222         </joint>
-223      <link name="tag2">
-224           <inertial>
-225               <mass value="0.0001" />
-226               <origin xyz="0 0 0" />
-227               <inertia ixx="0.0001" ixy="0.0" ixz="0.0"
-228                        iyy="0.0001" iyz="0.0"
-229                        izz="0.0001" />
-230           </inertial>
-231         </link>
-232         <joint name="yeet_tag2_joint" type="fixed">
-233                 <origin xyz="0 0.105 0" rpy="${pi * 1.5} ${pi} 0"/>
-234                 <parent link="yeet_box"/>
-235                 <child link="tag2"/>
-236         </joint>
-237      <link name="tag3">
-238           <inertial>
-239               <mass value="0.0001" />
-240               <origin xyz="0 0 0" />
-241               <inertia ixx="0.0001" ixy="0.0" ixz="0.0"
-242                        iyy="0.0001" iyz="0.0"
-243                        izz="0.0001" />
-244           </inertial>
-245         </link>
-246         <joint name="yeet_tag3_joint" type="fixed">
-247                 <origin xyz="0.105 0 0" rpy="${pi * 0.5} 0 ${pi * 0.5}"/>
-248                 <parent link="yeet_box"/>
-249                 <child link="tag3"/>
-250         </joint>
+     <link name="yeet_box">
+          <visual>
+            <geometry>
+              <box size="0.21 0.21 0.21" />
+            </geometry>
+            <material name="Blue" />
+          </visual>
+          <inertial>
+              <mass value="0.0001" />
+              <origin xyz="0 0 0" />
+              <inertia ixx="0.0001" ixy="0.0" ixz="0.0"
+                       iyy="0.0001" iyz="0.0"
+                       izz="0.0001" />
+          </inertial>
+        </link>
+        <joint name="base_yeet_joint" type="fixed">
+                <origin xyz="-0.075 0 1.28" rpy="0 0 0"/>
+                <parent link="base_link"/>
+                <child link="yeet_box"/>
+        </joint>
+     <link name="tag0">
+          <inertial>
+              <mass value="0.0001" />
+              <origin xyz="0 0 0" />
+              <inertia ixx="0.0001" ixy="0.0" ixz="0.0"
+                       iyy="0.0001" iyz="0.0"
+                       izz="0.0001" />
+          </inertial>
+        </link>
+        <joint name="yeet_tag0_joint" type="fixed">
+                <origin xyz="0 -0.105 0" rpy="${pi*0.5} 0 0"/>
+                <parent link="yeet_box"/>
+                <child link="tag0"/>
+        </joint>
+     <link name="tag1">
+          <inertial>
+              <mass value="0.0001" />
+              <origin xyz="0 0 0" />
+              <inertia ixx="0.0001" ixy="0.0" ixz="0.0"
+                       iyy="0.0001" iyz="0.0"
+                       izz="0.0001" />
+          </inertial>
+        </link>
+        <joint name="yeet_tag1_joint" type="fixed">
+                <origin xyz="-0.105 0 0" rpy="${pi*0.5} 0 ${pi*1.5}"/>
+                <parent link="yeet_box"/>
+                <child link="tag1"/>
+        </joint>
+     <link name="tag2">
+          <inertial>
+              <mass value="0.0001" />
+              <origin xyz="0 0 0" />
+              <inertia ixx="0.0001" ixy="0.0" ixz="0.0"
+                       iyy="0.0001" iyz="0.0"
+                       izz="0.0001" />
+          </inertial>
+        </link>
+        <joint name="yeet_tag2_joint" type="fixed">
+                <origin xyz="0 0.105 0" rpy="${pi * 1.5} ${pi} 0"/>
+                <parent link="yeet_box"/>
+                <child link="tag2"/>
+        </joint>
+     <link name="tag3">
+          <inertial>
+              <mass value="0.0001" />
+              <origin xyz="0 0 0" />
+              <inertia ixx="0.0001" ixy="0.0" ixz="0.0"
+                       iyy="0.0001" iyz="0.0"
+                       izz="0.0001" />
+          </inertial>
+        </link>
+        <joint name="yeet_tag3_joint" type="fixed">
+                <origin xyz="0.105 0 0" rpy="${pi * 0.5} 0 ${pi * 0.5}"/>
+                <parent link="yeet_box"/>
+                <child link="tag3"/>
+        </joint>
 <!-- Kinect Depth Sensor  -->
      <link name="camera_link">
